Commit message: updates

File: legged_gym/experiment/mesh_generation/parkour_meshes/whole_map/rectangular_prism_bumps.urdf (robot description, URDF)
Before this commit: robot rectangular_prism_bumps, 1 links, 0 joints
Links:
- link _name: geometry visual mesh filename=rectangular_prism_bumps.obj scale=1 1 1
